File: kicad/plate/key_matrix.kicad_sch (KiCad schematic)
At the start: 46 parts, among them SW1 EC_SW

Commit message: should be ok for proto order
Parts:
- SW1: footprint capacitive_sensors:ecs_plate_cut_1U_14x14mm -> (none)
